File: Aislador_USB/Aislador_USB.kicad_pcb (KiCad board)
At the start: 2 copper layers, 66 x 23.5 mm, 21 parts, among them U1 USBLC6-2SC6, U2 ADUM3160BRWZ-RL, U3 TEA1-0505, U4 USBLC6-2SC6

Commit message: 250425
Parts:
- added H1: MountingHole, MountingHole:MountingHole_3.2mm_M3, F.Cu at (119.5, 81.8)
- added H2: MountingHole, MountingHole:MountingHole_3.2mm_M3, F.Cu at (173.1, 81.8)
- added H3: MountingHole, MountingHole:MountingHole_3.2mm_M3, F.Cu at (119.5, 105.1)
- added H4: MountingHole, MountingHole:MountingHole_3.2mm_M3, F.Cu at (173.1, 105.1)
Other:
- board size 66 x 23.5 mm -> 62.8 x 32.1 mm
