File: Aislador_USB/Aislador_USB.kicad_sch (KiCad schematic)
At the start: 21 parts, among them U1 USBLC6-2SC6, U2 ADUM3160BRWZ-RL, U3 TEA1-0505, U4 USBLC6-2SC6

Commit message: 250425
Parts:
- added H1, H2, H3, H4: MountingHole, MountingHole:MountingHole_3.2mm_M3, symbol Mechanical:MountingHole
